File: electronics/rev_b/feedback/output_feedback.kicad_sch (KiCad schematic)
At the start: 10 parts, among them J1 POST-SWITCH L, J2 POST-SWITCH N, J3 3V3 / GND / OUT_N, U1 ACPL-K376-560E

Commit message: refactor: unify project and CARBENTRA branding
Other:
- title: CarbonMirror Rev B output detector -> CARBENTRA Rev B output detector
