File: electronics/rev_b/integrated/integrated.kicad_sch (KiCad schematic)
At the start: 3 parts, among them Y201 ASV-8.192MHZ-LC-S-T / candida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

Commit message: refactor: unify project and CARBENTRA branding
Other:
- note added: "CARBENTRA / CARBENTRA-P16-EVT-B INTEGRATED ELECTRICAL SOURCE"
- note removed: "CARBENTRA / CM-S16-EVT-B INTEGRATED ELECTRICAL SOURCE"
- title: CARBENTRA CM-S16-EVT-B integrated source -> CARBENTRA CARBENTRA-P16-EVT-B integrated source
