File: electronics/rev_b/integrated/integrated_meter.kicad_sch (KiCad schematic)
At the start: 34 parts, among them J201 PROTECTED LINE + NEUTRAL INPUT, U201 ATM90E26-YU, U202 ISO6741DWR

Commit message: refactor: unify project and CARBENTRA branding
Other:
- note added: "CARBENTRA REV B - METER - DEVELOPMENT / ENERGIZATION HOLD"
- note removed: "CARBONMIRROR REV B - METER - DEVELOPMENT / ENERGIZATION HOLD"
