File: electronics/rev_b/integrated/integrated_power_baseline.kicad_pcb (KiCad board)
At the start: 4 copper layers, 100 x 85 mm, 105 parts, among them J102 SWITCHED OUT - HOLD, J104 DEBUG - MAINS DISCONNECTED, J201 PROTECTED LINE + NEUTRAL INPUT, J403 SENSOR HARNESS, K101 RT314005 / 5V, Q101 AO3400A, Q401 AO3401A, Q402 MMBT3904, Q403 MMBT3904, SW101 LOCAL BUTTON, SW401 MANUAL REARM, U101 ESP32-C3-WROOM-02U-N4, U102 AP63203WU-7, U103 TMP102AIDRLR, U201 ATM90E26-YU, U202 ISO6741DWR, U301 ACPL-K376-560E, U402 SN74LVC1G17DBVR, U403 TPS3808G30DBVR, U404 SN74LVC1G74DCUR, U405 SN74LVC1G17DBVR, U406 SN74LVC1G17DBVR, Y201 ASV-8.192MHZ-LC-S-T / candida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

Commit message: refactor: unify project and CARBENTRA branding
Other:
- board text added: "CARBENTRA INTEGRATED B"
- board text removed: "CARBONMIRROR INTEGRATED B"
