File: electronics/rev_b/meter/meter.kicad_sch (KiCad schematic)
At the start: 39 parts, among them J1 PROTECTED L / TO RELAY, J2 N SENSE / NC, J3 CONTROLLER - ISOLATED, U1 ATM90E26-YU, U2 ISO6741DWR, Y1 8.192MHz CL18pF

Commit message: refactor: unify project and CARBENTRA branding
Other:
- note added: "CARBENTRA REV B - METER - DEVELOPMENT / ENERGIZATION HOLD"
- note removed: "CARBONMIRROR REV B - METER - DEVELOPMENT / ENERGIZATION HOLD"
- title: CarbonMirror REV B isolated metering -> CARBENTRA REV B isolated metering
