File: electronics/rev_b/thermal/thermal_interlock.kicad_sch (KiCad schematic)
At the start: 35 parts, among them J1 MAIN 4-WIRE COIL INTERLOCK, J3 SENSOR HARNESS, J4 SENSOR PIGTAIL, Q1 AO3401A, Q2 MMBT3904, Q3 MMBT3904, SW1 MANUAL REARM, U1 TMP302BDRLR, U2 SN74LVC1G17DBVR, U3 TPS3808G30DBVR, U4 SN74LVC1G74DCUR, U5 SN74LVC1G17DBVR, U6 SN74LVC1G17DBVR

Commit message: refactor: unify project and CARBENTRA branding
Other:
- title: CarbonMirror Rev B hardware thermal interlock -> CARBENTRA Rev B hardware thermal interlock
