File: electronics/rev_b/integrated/validation/rule_controls/supported.kicad_pcb (KiCad board)
At the start: 4 copper layers, 20 x 15 mm, 2 parts

Commit message: Localize and verify the current CARBENTRA Plug engineering toolchain
Validated source tree: 828281c98571813db5d4ddcfd2d92c1c9937963d. Preserve prior public main history. Complete delivery/local evolution and original edits remain in local archive and preserve branches.
Changed lines of the file:
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@@
 (kicad_pcb
-	(version 20241229)
+	(version 20260206)
 	(generator "pcbnew")
-	(generator_version "9.0")
+	(generator_version "10.0")
 	(general
 		(thickness 1.6)
@@
 		(pad_to_mask_clearance 0)
 		(allow_soldermask_bridges_in_footprints no)
-		(tenting front back)
+		(tenting
+			(front yes)
+			(back yes)
+		)
+		(covering
+			(front no)
+			(back no)
+		)
+		(plugging
+			(front no)
+			(back no)
+		)
+		(capping no)
+		(filling no)
 		(pcbplotparams
 			(layerselection 0x00000000_00000000_55555555_5755f5ff)
@@
 			(usegerberadvancedattributes yes)
 			(creategerberjobfile yes)
-			(dashed_line_dash_ratio 12.000000)
-			(dashed_line_gap_ratio 3.000000)
+			(dashed_line_dash_ratio 12)
+			(dashed_line_gap_ratio 3)
 			(svgprecision 4)
 			(plotframeref no)
 			(mode 1)
 			(useauxorigin no)
-			(hpglpennumber 1)
-			(hpglpenspeed 20)
-			(hpglpendiameter 15.000000)
 			(pdf_front_fp_property_popups yes)
 			(pdf_back_fp_property_popups yes)
@@
 		)
 	)
-	(net 0 "")
-	(net 1 "HOT_TEST")
-	(net 2 "ISO_TEST")
 	(footprint ""
 		(layer "F.Cu")
@@
 				(font
 					(size 1.27 1.27)
-					(thickness 0.15)
 				)
 			)
@@
 				(font
 					(size 1.27 1.27)
-					(thickness 0.15)
 				)
 			)
@@
 				(font
 					(size 1.27 1.27)
-					(thickness 0.15)
 				)
 			)
@@
 				(font
 					(size 1.27 1.27)
-					(thickness 0.15)
-				)
-			)
-		)
+				)
+			)
+		)
+		(duplicate_pad_numbers_are_jumpers no)
 		(pad "1" smd rect
 			(at 0 0)
 			(size 1 1)
 			(layers "F.Cu")
-			(net 1 "HOT_TEST")
+			(net "HOT_TEST")
 			(thermal_bridge_angle 45)
 		)
@@
 				(font
 					(size 1.27 1.27)
-					(thickness 0.15)
 				)
 			)
@@
 				(font
 					(size 1.27 1.27)
-					(thickness 0.15)
 				)
 			)
@@
 				(font
 					(size 1.27 1.27)
-					(thickness 0.15)
 				)
 			)
@@
 				(font
 					(size 1.27 1.27)
-					(thickness 0.15)
-				)
-			)
-		)
+				)
+			)
+		)
+		(duplicate_pad_numbers_are_jumpers no)
 		(pad "1" smd rect
 			(at 0 0)
 			(size 1 1)
 			(layers "F.Cu")
-			(net 2 "ISO_TEST")
+			(net "ISO_TEST")
 			(thermal_bridge_angle 45)
 		)
@@
 	)
 	(gr_line
+		(start 5 20)
+		(end 5 5)
+		(stroke
+			(width 0.05)
+			(type default)
+		)
+		(layer "Edge.Cuts")
+	)
+	(gr_line
 		(start 25 5)
 		(end 25 20)
@@
 		(stroke
 			(width 0.05)
-			(type default)
-		)
-		(layer "Edge.Cuts")
-	)
-	(gr_line
-		(start 5 20)
-		(end 5 5)
-		(stroke
-			(width 0.05)
